File: esp32_iot_board/_autosave-esp32_iot_board.kicad_pcb (KiCad board)
At the start: 2 copper layers, 100 x 100 mm, 62 parts, among them J1 USB_C_Receptacle_USB2.0, J2 Conn_01x04, J3 Screw_Terminal_01x03, J4 Screw_Terminal_01x08, J5 Screw_Terminal_01x02, J6 Conn_02x05_Odd_Even, K1 RT314A05, Q1 UMH3N, Q2 BC817, SW1 SW_SPST, U1 ESP32-WROOM-32D, U2 USBLC6-2P6, U3 CP2104, U4 Si7020-A20, U5 74AHCT245, U6 TLV1117LV-3.3

Commit message: 2.06h
Parts:
- moved C7 160.5 mm to (105.9, 97.2), turned to -90 degrees
- moved C9 155.1 mm to (116.6, 67.0), turned to 90 degrees
- moved R1 154.9 mm to (98.9, 94.9), turned to -90 degrees
- moved C14 154.7 mm to (123.7, 63.5)
- moved C15 154.7 mm to (123.7, 66.8)
- moved R2 151.8 mm to (101.3, 94.9), turned to -90 degrees
- moved C8 145.1 mm to (121.7, 93.1)
- moved R10 141.0 mm to (120.3, 113.1)
- moved R8 141.0 mm to (120.3, 106.6)
- moved R9 141.0 mm to (120.3, 109.8)
- moved R7 138.9 mm to (116.6, 72.6), turned to 90 degrees
- moved R6 138.5 mm to (119.8, 87.9), turned to 90 degrees
- moved R11 137.2 mm to (123.4, 58.7)
- moved R17 95.7 mm to (171.6, 76.2)
- moved R18 95.7 mm to (171.6, 79.5)
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